Commit message: camilocommit

File: urdf/to.urdf (robot description, URDF)
Before this commit: robot anymal, 22 links, 21 joints
Links:
- removed link LF_ADAPTER
- removed link LF_FOOT
- removed link LF_SHANK
- removed link LF_THIGH
- removed link LH_ADAPTER
- removed link LH_FOOT
- removed link LH_HIP
- removed link LH_SHANK
- removed link LH_THIGH
- removed link RF_ADAPTER
- removed link RF_FOOT
- removed link RF_SHANK
- removed link RF_THIGH
- removed link RH_ADAPTER
- removed link RH_FOOT
- removed link RH_HIP
- removed link RH_SHANK
- removed link RH_THIGH
- added link LF_FLX1, mass 0.263; collision box size=0.061 0.060 0.181912; visual mesh filename=package://to_description/meshes/flex_1_fl.dae scale=0.001 0.001 0.001
- added link LF_FLX2, mass 0.263; collision box size=0.021 0.021 0.146; visual mesh filename=package://to_description/meshes/tibia.dae scale=0.001 0.001 0.001
- added link LF_FT, mass 0.263; collision sphere radius=0.0278; visual mesh filename=package://to_description/meshes/foot.dae scale=0.001 0.001 0.001
- added link LR_FLX1, mass 0.263; collision box size=0.061 0.060 0.181912; visual mesh filename=package://to_description/meshes/flex_1_fl.dae scale=0.001 0.001 0.001
- added link LR_FLX2, mass 0.263; collision box size=0.021 0.021 0.146; visual mesh filename=package://to_description/meshes/tibia.dae scale=0.001 0.001 0.001
- added link LR_FT, mass 0.263; collision sphere radius=0.0278; visual mesh filename=package://to_description/meshes/foot.dae scale=0.001 0.001 0.001
- added link LR_HIP, mass 0.255; collision box size=0.181912 0.061 0.060; visual mesh filename=package://to_description/meshes/ab_left_rear.dae scale=0.001 0.001 0.001
- added link RF_FLX1, mass 0.263; collision box size=0.061 0.060 0.181912; visual mesh filename=package://to_description/meshes/flex_1_fr.dae scale=0.001 0.001 0.001
- added link RF_FLX2, mass 0.263; collision box size=0.021 0.021 0.146; visual mesh filename=package://to_description/meshes/tibia_rigth.dae scale=0.001 0.001 0.001
- added link RF_FT, mass 0.263; collision sphere radius=0.0278; visual mesh filename=package://to_description/meshes/foot.dae scale=0.001 0.001 0.001
- added link RR_FLX1, mass 0.263; collision box size=0.061 0.060 0.181912; visual mesh filename=package://to_description/meshes/flex_1_fr.dae scale=0.001 0.001 0.001
- added link RR_FLX2, mass 0.263; collision box size=0.021 0.021 0.146; visual mesh filename=package://to_description/meshes/tibia_rigth.dae scale=0.001 0.001 0.001
- added link RR_FT, mass 0.263; collision sphere radius=0.0278; visual mesh filename=package://to_description/meshes/foot.dae scale=0.001 0.001 0.001
- added link RR_HIP, mass 0.255; collision box size=0.181912 0.061 0.060; visual mesh filename=package://to_description/meshes/ab_rrear.dae scale=0.001 0.001 0.001
- link LF_HIP: mass 1.42462064 -> 0.272; geometry collision box size=0.181912 0.061 0.060; visual mesh filename=package://to_description/meshes/ab_lf.dae scale=0.001 0.001 0.001
- link RF_HIP: mass 1.42462064 -> 0.255; geometry collision box size=0.181912 0.061 0.060; visual mesh filename=package://to_description/meshes/ab_fr_simplify.dae scale=0.001 0.001 0.001
- link base: geometry collision box size=0.600 0.255 0.01; visual mesh filename=package://to_description/meshes/chasis_abs_simply3.dae scale=0.001 0.001 0.001
- link base_inertia: mass 16.793507758 -> 0.293
Joints:
- removed joint LF_ADAPTER_TO_FOOT
- removed joint LF_HAA
- removed joint LF_HFE
- removed joint LF_KFE
- removed joint LF_SHANK_TO_ADAPTER
- removed joint LH_ADAPTER_TO_FOOT
- removed joint LH_HAA
- removed joint LH_HFE
- removed joint LH_KFE
- removed joint LH_SHANK_TO_ADAPTER
- removed joint RF_ADAPTER_TO_FOOT
- removed joint RF_HAA
- removed joint RF_HFE
- removed joint RF_KFE
- removed joint RF_SHANK_TO_ADAPTER
- removed joint RH_ADAPTER_TO_FOOT
- removed joint RH_HAA
- removed joint RH_HFE
- removed joint RH_KFE
- removed joint RH_SHANK_TO_ADAPTER
- added joint LF_ABD: type revolute, parent base, child LF_HIP, origin xyz=0.055657 0.105030 0.042319 rpy=0.0 0.0 0.0, axis 1 0 0, limit lower=-0.42 upper=1.14 effort=80 velocity=15
- added joint LF_FF2: type revolute, parent LF_FLX1, child LF_FLX2, origin xyz=0.0 0.064575 -0.1534 rpy=0.0 0.0 0.0, axis 0 1 0, limit lower=-1.62 upper=1.62 effort=80 velocity=15
- added joint LF_FT_FX: type fixed, parent LF_FLX2, child LF_FT, origin xyz=0.0 0.0304 -0.192206 rpy=0 0 0
- added joint LF_HF1: type revolute, parent LF_HIP, child LF_FLX1, origin xyz=0.204912 0.014725 0.0 rpy=0.0 0.0 0.0, axis 0 1 0, limit lower=-1.62 upper=1.62 effort=80 velocity=15
- added joint LR_ABD: type revolute, parent base, child LR_HIP, origin xyz=-0.102751 0.105030 0.041319 rpy=0.0 0.0 0.0, axis 1 0 0, limit lower=-0.42 upper=1.14 effort=80 velocity=15
- added joint LR_FF2: type revolute, parent LR_FLX1, child LR_FLX2, origin xyz=0.0 0.064575 -0.1534 rpy=0.0 0.0 0.0, axis 0 1 0, limit lower=-1.62 upper=1.62 effort=80 velocity=15
- added joint LR_FT_FX: type fixed, parent LR_FLX2, child LR_FT, origin xyz=0.0 0.0304 -0.192206 rpy=0 0 0
- added joint LR_HF1: type revolute, parent LR_HIP, child LR_FLX1, origin xyz=-0.157912 0.014725 0.0 rpy=0.0 0.0 0.0, axis 0 1 0, limit lower=-1.62 upper=1.62 effort=80 velocity=15
- added joint RF_ABD: type revolute, parent base, child RF_HIP, origin xyz=0.102751 -0.105030 0.041319 rpy=0.0 0.0 0.0, axis 1 0 0, limit lower=-0.42 upper=1.14 effort=80 velocity=15
- added joint RF_FF2: type revolute, parent RF_FLX1, child RF_FLX2, origin xyz=0.0 -0.064575 -0.1534 rpy=0.0 0.0 0.0, axis 0 1 0, limit lower=-1.62 upper=1.62 effort=80 velocity=15
- added joint RF_FT_FX: type fixed, parent RF_FLX2, child RF_FT, origin xyz=0.0 -0.0304 -0.192206 rpy=0 0 0
- added joint RF_HF1: type revolute, parent RF_HIP, child RF_FLX1, origin xyz=0.157912 -0.014725 0.0 rpy=0.0 0.0 0.0, axis 0 1 0, limit lower=-1.62 upper=1.62 effort=80 velocity=15
- added joint RR_ABD: type revolute, parent base, child RR_HIP, origin xyz=-0.055657 -0.105030 0.041319 rpy=0.0 0.0 0.0, axis 1 0 0, limit lower=-0.42 upper=1.14 effort=80 velocity=15
- added joint RR_FF2: type revolute, parent RR_FLX1, child RR_FLX2, origin xyz=0.0 -0.064575 -0.1534 rpy=0.0 0.0 0.0, axis 0 1 0, limit lower=-1.62 upper=1.62 effort=80 velocity=15
- added joint RR_FT_FX: type fixed, parent RR_FLX2, child RR_FT, origin xyz=0.0 -0.0304 -0.192206 rpy=0 0 0
- added joint RR_HF1: type revolute, parent RR_HIP, child RR_FLX1, origin xyz=-0.204912 -0.014725 0.0 rpy=0.0 0.0 0.0, axis 0 1 0, limit lower=-1.62 upper=1.62 effort=80 velocity=15
